Commit message: Added Moveit - More work needed to be done

File: install/excavator_description/share/excavator_description/urdf/excavator.urdf.xacro (robot description, xacro)
@@ -7,9 +7,10 @@
     <!-- Include ros2_control Plugins -->
     <xacro:include filename="$(find excavator_description)/urdf/excavator_ros2_control.xacro" />
+  <link name="world"/>
   <link
     name="base_link">
     <inertial>
       <origin
-        xyz="-3.05023976636919E-16 -1.20579956142935 -0.755810436649642"
+        xyz="0 0 1.29"
         rpy="0 0 0" />
       <mass
@@ -25,5 +26,5 @@
     <visual>
       <origin
-        xyz="0 0 0"
+        xyz="0 0 1.29"
         rpy="0 0 0" />
       <geometry>
@@ -39,5 +40,5 @@
     <collision>
       <origin
-        xyz="0 0 0"
+        xyz="0 0 1.29"
         rpy="0 0 0" />
       <geometry>
@@ -51,5 +52,5 @@
     <inertial>
       <origin
-        xyz="-0.0572240980964203 -1.43061378500035 0.653734550513117"
+        xyz="-0.0572240980964203 -1.43061378500035 1.023734551"
         rpy="0 0 0" />
       <mass
@@ -65,5 +66,5 @@
     <visual>
       <origin
-        xyz="0 0 0"
+        xyz="0 0 1.023734551"
         rpy="0 0 0" />
       <geometry>
@@ -79,5 +80,5 @@
     <collision>
       <origin
-        xyz="0 0 0"
+        xyz="0 0 1.023734551"
         rpy="0 0 0" />
       <geometry>
@@ -279,3 +280,8 @@
       velocity="100" />
   </joint>
+  <joint name="virtual_joint" type="fixed">
+        <parent link="world"/>
+        <child link="base_link"/>
+        <origin xyz="0 0 0" rpy="0 0 0"/>
+    </joint>
 </robot>
